Commit message: fix airplane.urdf

File: hot/data/assets/urdf/airplane/airplane.urdf (robot description, URDF)
Before this commit: robot airplane, 1 links, 0 joints
Links:
- link base_link: geometry collision mesh filename=top_watertight_tiny.stl scale=1 1 1; visual mesh filename=top_watertight_tiny.stl scale=1 1 1
